File: StudioClock.sch (KiCad schematic (older format))
At the start: 80 parts, among them J1 CONN_01X16, J2 CONN_01X16, U1 7SEGMENTS, U2 7SEGMENTS, U3 7SEGMENTS, U4 7SEGMENTS

Commit message: script runs, updated symbols and footprints
Parts:
- D1, D10, D11, D12, D13, D14, D15, D16, D17, D18, D19, D2, D20, D21, D22, D23, D24, D25, D26, D27, D28, D29, D3, D30, D31, D32, D33, D34, D35, D36, D37, D38, D39, D4, D40, D41, D42, D43, D44, D45, D46, D47, D48, D49, D5, D50, D51, D52, D53, D54, D55, D56, D57, D58, D59, D6, D60, D61, D62, D63, D64, D65, D66, D67, D68, D69, D7, D70, D71, D72, D73, D74, D8, D9: footprint LEDs:LED_0805 -> LED_SMD:LED_0805_2012Metric; symbol LED -> StudioClock-rescue:LED
- J1, J2: footprint Pin_Headers:Pin_Header_Straight_1x16_Pitch2.54mm_SMD_Pin1Left -> Connector_PinHeader_2.54mm:PinHeader_1x16_P2.54mm_Vertical_SMD_Pin1Left; symbol CONN_01X16 -> Connector_Generic:Conn_01x16
- U1, U2, U3, U4: footprint (none) -> Display_7Segment:7SEGMENT-LED__HDSM531_HDSM533_SMD; symbol 7SEGMENTS -> StudioClock-rescue:7SEGMENTS
Connections:
- wire segments 264 -> 392

Commit message: executed and cleaned up files, added README
Parts:
- D1, D10, D11, D12, D13, D14, D15, D16, D17, D18, D19, D2, D20, D21, D22, D23, D24, D25, D26, D27, D28, D29, D3, D30, D31, D32, D33, D34, D35, D36, D37, D38, D39, D4, D40, D41, D42, D43, D44, D45, D46, D47, D48, D49, D5, D50, D51, D52, D53, D54, D55, D56, D57, D58, D59, D6, D60, D61, D62, D63, D64, D65, D66, D67, D68, D69, D7, D70, D71, D72, D73, D74, D8, D9: symbol StudioClock-rescue:LED -> Device:LED
